File: ArduinoUnoR4Shield.kicad_sch (KiCad schematic)
At the start: 11 parts, among them U1 OFF, U2 Analog_1, U3 Analog_2, U4 ESP32-S3, U5 ICSP, U6 Digital_1, U7 Digital_2

Commit message: Updated Titles
Other:
- title: Arduino UNO R4 Shield Template SCH -> Arduino UNO R4 Proto Shield  Template SCH
Changed lines of the file:
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@@
   (paper "A4")
   (title_block
-    (title "Arduino UNO R4 Shield Template SCH")
+    (title "Arduino UNO R4 Proto Shield  Template SCH")
     (date "2023-07-13")
     (rev "1.0")
